Commit message: Implement working research baseline v0.1 with safety monitor and task sequence

File: ros2_ws/src/peg_in_hole_description/urdf/peg_in_hole_task.urdf.xacro (robot description, xacro)
@@ -11,5 +11,5 @@
     <parent link="world"/>
     <child link="target_hole_frame"/>
-    <origin xyz="0.60 0.0 0.81" rpy="0 0 0"/>
+    <origin xyz="0.52 -0.20 0.81" rpy="0 0 0"/>
   </joint>
   <link name="peg_tip"/>
