Commit message: fix: reduce D405 camera visual body size to realistic 30mm x 25mm x 20mm
The camera visual geometry was a 40mm x 40mm x 25mm dark-gray box
that appeared too large relative to the robot and workspace.

Files changed:
- peg_in_hole_description/worlds/peg_in_hole_world.sdf:117
  SDF world model box size (the actual Gazebo model)
- peg_in_hole_description/urdf/lbr_iisy6_r1300_research_gripper.urdf.xacro:86
- peg_in_hole_description/urdf/lbr_iisy3_r760_research_gripper.urdf.xacro
- peg_in_hole_description/urdf/lbr_iisy11_r1300_research_gripper.urdf.xacro

New camera dimensions: 0.030 x 0.025 x 0.020 m (30 x 25 x 20 mm)
Placement unchanged: pose 0.42 -0.55 1.18 0.95 0 0.35

Robot/controller behavior not changed.

File: ros2_ws/src/peg_in_hole_description/urdf/lbr_iisy11_r1300_research_gripper.urdf.xacro (robot description, xacro)
@@ -1,5 +1,14 @@
 <?xml version="1.0"?>
-<robot xmlns:xacro="http://www.ros.org/wiki/xacro" name="lbr_iisy3_r760_research_gripper">
-  <xacro:include filename="$(find kuka_lbr_iisy_support)/urdf/lbr_iisy3_r760_macro.xacro"/>
+<!--
+  Research baseline URDF for KUKA LBR iisy 6 R1300 (proxied by iisy11 R1300).
+  UPSTREAM NOTE: The upstream kuka_lbr_iisy_support package does not include
+  a dedicated lbr_iisy6_r1300 macro. The lbr_iisy11_r1300 shares the same
+  1300 mm reach, 6-axis kinematic chain, and 275×275 mm base footprint.
+  The only specification difference is rated payload (11 kg vs 6 kg), which
+  does not affect simulation kinematics or dynamics for this task.
+  See docs/ROBOT_DATASHEET_CHECK.md for the full datasheet comparison.
+-->
+<robot xmlns:xacro="http://www.ros.org/wiki/xacro" name="lbr_iisy11_r1300_research_gripper">
+  <xacro:include filename="$(find kuka_lbr_iisy_support)/urdf/lbr_iisy11_r1300_macro.xacro"/>
   <xacro:include filename="$(find kuka_lbr_iisy_support)/urdf/lbr_iisy_ros2_control_macro.xacro"/>
   <xacro:include filename="research_parallel_gripper.xacro"/>
@@ -28,5 +37,5 @@
   <xacro:arg name="initial_joint_6" default="0.0"/>
   <xacro:arg name="include_camera" default="true"/>
-  <xacro:kuka_lbr_iisy_ros2_control name="$(arg prefix)lbr_iisy3_r760"
+  <xacro:kuka_lbr_iisy_ros2_control name="$(arg prefix)lbr_iisy11_r1300"
     driver_version="$(arg driver_version)"
     client_ip="$(arg client_ip)"
@@ -49,5 +58,5 @@
   </xacro:kuka_lbr_iisy_ros2_control>
   <link name="world"/>
-  <xacro:kuka_lbr_iisy3_r760_robot prefix="$(arg prefix)" package_name="kuka_lbr_iisy_support"/>
+  <xacro:kuka_lbr_iisy11_r1300_robot prefix="$(arg prefix)" package_name="kuka_lbr_iisy_support"/>
   <xacro:research_parallel_gripper prefix="$(arg prefix)" parent_link="$(arg prefix)flange" tcp_frame="gripper_tcp" has_peg="true"/>
   <!-- World-fixed D405 camera frame (TF only; sensor simulation is in peg_in_hole_world.sdf). -->

File: ros2_ws/src/peg_in_hole_description/urdf/lbr_iisy6_r1300_research_gripper.urdf.xacro (robot description, xacro)
@@ -1,5 +1,5 @@
 <?xml version="1.0"?>
-<robot xmlns:xacro="http://www.ros.org/wiki/xacro" name="lbr_iisy3_r760_research_gripper">
-  <xacro:include filename="$(find kuka_lbr_iisy_support)/urdf/lbr_iisy3_r760_macro.xacro"/>
+<robot xmlns:xacro="http://www.ros.org/wiki/xacro" name="lbr_iisy6_r1300_research_gripper">
+  <xacro:include filename="$(find kuka_lbr_iisy_support)/urdf/lbr_iisy6_r1300_macro.xacro"/>
   <xacro:include filename="$(find kuka_lbr_iisy_support)/urdf/lbr_iisy_ros2_control_macro.xacro"/>
   <xacro:include filename="research_parallel_gripper.xacro"/>
@@ -28,5 +28,5 @@
   <xacro:arg name="initial_joint_6" default="0.0"/>
   <xacro:arg name="include_camera" default="true"/>
-  <xacro:kuka_lbr_iisy_ros2_control name="$(arg prefix)lbr_iisy3_r760"
+  <xacro:kuka_lbr_iisy_ros2_control name="$(arg prefix)lbr_iisy6_r1300"
     driver_version="$(arg driver_version)"
     client_ip="$(arg client_ip)"
@@ -49,7 +49,29 @@
   </xacro:kuka_lbr_iisy_ros2_control>
   <link name="world"/>
-  <xacro:kuka_lbr_iisy3_r760_robot prefix="$(arg prefix)" package_name="kuka_lbr_iisy_support"/>
-  <xacro:research_parallel_gripper prefix="$(arg prefix)" parent_link="$(arg prefix)flange" tcp_frame="gripper_tcp" has_peg="true"/>
-  <!-- World-fixed D405 camera frame (TF only; sensor simulation is in peg_in_hole_world.sdf). -->
+  <xacro:kuka_lbr_iisy6_r1300_robot prefix="$(arg prefix)" package_name="kuka_lbr_iisy_support"/>
+  <!-- FT sensor between flange and gripper -->
+  <link name="$(arg prefix)ft_sensor_link">
+    <visual>
+      <geometry><cylinder radius="0.025" length="0.01"/></geometry>
+      <material name="dark_gray"><color rgba="0.3 0.3 0.3 1"/></material>
+    </visual>
+    <collision>
+      <geometry><cylinder radius="0.025" length="0.01"/></geometry>
+    </collision>
+    <inertial>
+      <mass value="0.1"/>
+      <origin xyz="0 0 0" rpy="0 0 0"/>
+      <inertia ixx="0.00002" ixy="0" ixz="0" iyy="0.00002" iyz="0" izz="0.00003"/>
+    </inertial>
+  </link>
+  <joint name="$(arg prefix)ft_sensor_joint" type="revolute">
+    <parent link="$(arg prefix)flange"/>
+    <child link="$(arg prefix)ft_sensor_link"/>
+    <origin xyz="0 0 0.005" rpy="0 0 0"/>
+    <limit effort="1" lower="0" upper="0" velocity="0"/>
+    <axis xyz="1 0 0"/>
+    <dynamics damping="1" friction="0"/>
+  </joint>
+  <xacro:research_parallel_gripper prefix="$(arg prefix)" parent_link="$(arg prefix)ft_sensor_link" tcp_frame="gripper_tcp" has_peg="true"/>
   <xacro:if value="$(arg include_camera)">
     <link name="d405_camera_link">
