Commit message: Validate iisy6 cell model consistency

File: ros2_ws/src/peg_in_hole_description/urdf/lbr_iisy6_r1300_research_gripper.urdf.xacro (robot description, xacro)
@@ -27,5 +27,5 @@
   <xacro:arg name="initial_joint_5" default="0.8"/>
   <xacro:arg name="initial_joint_6" default="0.0"/>
-  <xacro:arg name="include_camera" default="true"/>
+  <xacro:arg name="include_camera" default="false"/>
   <xacro:kuka_lbr_iisy_ros2_control name="$(arg prefix)lbr_iisy6_r1300"
     driver_version="$(arg driver_version)"
@@ -74,4 +74,7 @@
   </joint>
   <xacro:research_parallel_gripper prefix="$(arg prefix)" parent_link="$(arg prefix)ft_sensor_link" tcp_frame="gripper_tcp" has_peg="true"/>
+  <!-- The canonical Gazebo world owns the D405 sensor model. This optional
+       TF-only camera frame is disabled by default so URDF->SDF conversion of
+       the robot model stays self-contained. -->
   <xacro:if value="$(arg include_camera)">
     <link name="d405_camera_link">

File: ros2_ws/src/peg_in_hole_description/urdf/proposal_lbr_iisy6_r1300_cell.urdf.xacro (robot description, xacro)
@@ -1,3 +1,12 @@
 <?xml version="1.0"?>
+<!--
+  !!! DEPRECATED – CYLINDER-BASED PLACEHOLDER !!!
+  This file defines a fake cylinder robot with no kinematic accuracy.
+  It was used during early proposal validation (v1.x / early v2.x).
+  DO NOT use for any new work. Use instead:
+    peg_in_hole_description/urdf/lbr_iisy6_r1300_research_gripper.urdf.xacro
+  which includes the real mesh-based KUKA LBR iisy 6 R1300 description
+  with a research parallel gripper.
+-->
 <robot xmlns:xacro="http://www.ros.org/wiki/xacro" name="proposal_lbr_iisy6_r1300_cell">
   <link name="world"/>

File: ros2_ws/src/peg_in_hole_description/urdf/research_parallel_gripper.xacro (robot description, xacro)
@@ -1,5 +1,5 @@
 <?xml version="1.0"?>
 <robot xmlns:xacro="http://www.ros.org/wiki/xacro">
-  <xacro:macro name="research_parallel_gripper" params="prefix parent_link tcp_frame:=gripper_tcp">
+  <xacro:macro name="research_parallel_gripper" params="prefix parent_link tcp_frame:=gripper_tcp has_peg:=false">
     <xacro:property name="gripper_palm_x" value="0.080"/>
     <xacro:property name="gripper_palm_y" value="0.060"/>
@@ -98,4 +98,40 @@
       <origin xyz="0 0 ${gripper_tcp_z_offset}" rpy="0 0 0"/>
     </joint>
+    <xacro:if value="${has_peg}">
+      <xacro:property name="peg_radius" value="0.0125"/>
+      <xacro:property name="peg_length" value="0.11"/>
+      <xacro:property name="peg_center_z" value="${gripper_tcp_z_offset - peg_length / 2.0}"/>
+      <xacro:property name="peg_tip_z" value="${gripper_tcp_z_offset - peg_length}"/>
+      <material name="${prefix}peg_material">
+        <color rgba="0.70 0.72 0.74 1.0"/>
+      </material>
+      <link name="${prefix}grasped_peg">
+        <inertial>
+          <origin xyz="0 0 ${peg_center_z}" rpy="0 0 0"/>
+          <mass value="0.15"/>
+          <inertia ixx="0.000157" ixy="0.0" ixz="0.0" iyy="0.000157" iyz="0.0" izz="0.0000117"/>
+        </inertial>
+        <visual>
+          <origin xyz="0 0 ${peg_center_z}" rpy="0 0 0"/>
+          <geometry><cylinder radius="${peg_radius}" length="${peg_length}"/></geometry>
+          <material name="${prefix}peg_material"/>
+        </visual>
+        <collision>
+          <origin xyz="0 0 ${peg_center_z}" rpy="0 0 0"/>
+          <geometry><cylinder radius="${peg_radius}" length="${peg_length}"/></geometry>
+        </collision>
+      </link>
+      <joint name="${prefix}gripper_palm_to_grasped_peg" type="fixed">
+        <parent link="${prefix}gripper_palm"/>
+        <child link="${prefix}grasped_peg"/>
+        <origin xyz="0 0 0" rpy="0 0 0"/>
+      </joint>
+      <link name="${prefix}peg_tip"/>
+      <joint name="${prefix}grasped_peg_to_peg_tip" type="fixed">
+        <parent link="${prefix}grasped_peg"/>
+        <child link="${prefix}peg_tip"/>
+        <origin xyz="0 0 ${peg_tip_z}" rpy="0 0 0"/>
+      </joint>
+    </xacro:if>
   </xacro:macro>
 </robot>

Commit message: Raise FT mount effort limit

File: ros2_ws/src/peg_in_hole_description/urdf/lbr_iisy6_r1300_research_gripper.urdf.xacro (robot description, xacro)
@@ -50,5 +50,9 @@
   <link name="world"/>
   <xacro:kuka_lbr_iisy6_r1300_robot prefix="$(arg prefix)" package_name="kuka_lbr_iisy_support" collision_geometry="primitive"/>
-  <!-- FT sensor between flange and gripper -->
+  <!-- FT sensor between flange and gripper.
+       Gazebo's URDF->SDF conversion collapses fixed joints, so this zero-range
+       revolute joint is used only to preserve a named joint for the joint-level
+       force_torque sensor injected by spawn_robot_sdf.py. The high effort and
+       velocity limits avoid modeling the rigid sensor mount as a weak actuator. -->
   <link name="$(arg prefix)ft_sensor_link">
     <visual>
@@ -69,5 +73,5 @@
     <child link="$(arg prefix)ft_sensor_link"/>
     <origin xyz="0 0 0.005" rpy="0 0 0"/>
-    <limit effort="1" lower="0" upper="0" velocity="0"/>
+    <limit effort="10000" lower="0" upper="0" velocity="100"/>
     <axis xyz="1 0 0"/>
     <dynamics damping="1" friction="0"/>
